Commit message: 更新xwlurdf配置，调整初始位置、关节角度及物理参数

File: resources/robots/xwl/urdf/xwl.urdf (robot description, URDF)
Before this commit: robot xwl, 7 links, 6 joints
Links:
- link base_link: geometry collision mesh filename=../meshes/base_link.STL; visual mesh filename=../meshes/base_link.STL
- link ll1: geometry collision mesh filename=../meshes/ll1.STL; visual mesh filename=../meshes/ll1.STL
- link ll_0: geometry collision mesh filename=../meshes/ll_0.STL; visual mesh filename=../meshes/ll_0.STL
- link lw: geometry collision mesh filename=../meshes/lw.STL; visual mesh filename=../meshes/lw.STL
- link rl_0: geometry collision mesh filename=../meshes/rl_0.STL; visual mesh filename=../meshes/rl_0.STL
- link rl_1: geometry collision mesh filename=../meshes/rl_1.STL; visual mesh filename=../meshes/rl_1.STL
- link rw: geometry collision mesh filename=../meshes/rw.STL; visual mesh filename=../meshes/rw.STL
Joints:
- joint ll1_Joint: limit lower=0 upper=0 effort=0 velocity=0 -> lower=-0.94 upper=1.1 effort=10 velocity=1000
- joint ll_Joint0: axis 0 0 -1 -> 0 0 1; limit lower=0 upper=0 effort=0 velocity=0 -> lower=-0.57 upper=0.9 effort=10 velocity=1000
- joint lw_Joint: limit lower=0 upper=0 effort=0 velocity=0 -> lower=0 upper=0 effort=3 velocity=1000; type continuous -> revolute
- joint rl_Joint0: axis 0 0 -1 -> 0 0 1; limit lower=0 upper=0 effort=0 velocity=0 -> lower=-0.9 upper=0.57 effort=10 velocity=1000
- joint rl_Joint1: limit lower=0 upper=0 effort=0 velocity=0 -> lower=-1.1 upper=0.94 effort=10 velocity=1000
- joint rw_Joint: limit lower=0 upper=0 effort=0 velocity=0 -> lower=0 upper=0 effort=3 velocity=1000; type continuous -> revolute
