Commit message: 修复 xwl URDF 关节限位错误
- 轮关节 rw/lw_Joint 由 revolute(limit=[0,0]) 改为 continuous，
  之前 limit 锁死导致轮子完全无法转动，机器人只能靠腿挣扎
- 4 个腿关节的 limit 在默认关节角附近留出 0.5 rad 余量，
  之前默认值正好压在 limit 边界，spawn 瞬间触发关节限位反作用力 +
  PD 共振，造成腿在空中也高频抖动几厘米

Co-Authored-By: Claude Opus 4.7 (1M context) <noreply@anthropic.com>

File: resources/robots/xwl/urdf/xwl.urdf (robot description, URDF)
Before this commit: robot xwl, 7 links, 6 joints
Joints:
- joint ll1_Joint: limit lower=-0.94 upper=1.1 effort=10 velocity=1000 -> lower=-1.44 upper=1.1 effort=10 velocity=1000
- joint ll_Joint0: limit lower=-0.57 upper=0.9 effort=10 velocity=1000 -> lower=-0.57 upper=1.4 effort=10 velocity=1000
- joint lw_Joint: limit lower=0 upper=0 effort=3 velocity=1000 -> lower=-1000 upper=1000 effort=3 velocity=1000; type revolute -> continuous
- joint rl_Joint0: limit lower=-0.9 upper=0.57 effort=10 velocity=1000 -> lower=-1.4 upper=0.57 effort=10 velocity=1000
- joint rl_Joint1: limit lower=-1.1 upper=0.94 effort=10 velocity=1000 -> lower=-1.1 upper=1.44 effort=10 velocity=1000
- joint rw_Joint: limit lower=0 upper=0 effort=3 velocity=1000 -> lower=-1000 upper=1000 effort=3 velocity=1000; type revolute -> continuous
