Commit message: 重排 chuanliantui URDF 对齐 wl 关节轴约定,补齐惯量与电机参数
- base_link 转 x前/y左/z上,全部 joint axis 归一为 0 0 1,左右镜像,
  运动学与原始导出严格等价(FK 自检最大偏差 3e-16)
- lf0 零质量按左右对称件由 rf0 镜像补齐(m=1.0986kg)
- 腿关节 DM8009P effort=40/velocity=16.8;轮关节改装 M3508(减速比16.6)
  effort=3.9/velocity=58.4;轮转角限位解锁(wl 同款);关节限位数值未动

任务: T-20260823-01

Co-Authored-By: Claude Fable 5 <noreply@anthropic.com>

File: resources/robots/chuanliantui/urdf/chuanliantui.urdf (robot description, URDF)
Before this commit: robot chuanliantui, 7 links, 6 joints
Links:
- link lf0: mass 0 -> 1.0986
Joints:
- joint lf0: axis 0 -1 0 -> 0 0 1; limit lower=-100 upper=100 effort=0 velocity=0 -> lower=-100 upper=100 effort=40 velocity=16.8; origin xyz=-0.0114 0.02352 0.17857 rpy=-1.5708 0 0 -> xyz=0.0114 0.17857 0.02352 rpy=-1.5707926535897934 0 0
- joint lf1: axis 0 1 0 -> 0 0 1; limit lower=-0.77 upper=0.12 effort=0 velocity=0 -> lower=-0.77 upper=0.12 effort=40 velocity=16.8; origin xyz=-0.1651 -0.0115 -0.12977 rpy=0 0 0 -> xyz=0.1651 0.12977 0.0115 rpy=3.141592653589793 0 0
- joint lfwheel: axis 0 -1 0 -> 0 0 1; limit lower=0 upper=0 effort=0 velocity=0 -> effort=3.9 velocity=58.4; origin xyz=0.1651 -0.028 -0.18773 rpy=0 0 0 -> xyz=-0.1651 -0.18773 -0.028 rpy=3.141592653589793 0 0
- joint rf0: axis 0 1 0 -> 0 0 1; limit lower=-100 upper=100 effort=0 velocity=0 -> lower=-100 upper=100 effort=40 velocity=16.8; origin xyz=-0.0114 0.02352 -0.17693 rpy=-1.5708 0 0 -> xyz=0.0114 -0.17693 0.02352 rpy=1.5708 0 0
- joint rf1: axis 0 -1 0 -> 0 0 1; limit lower=-0.12 upper=0.77 effort=0 velocity=0 -> lower=-0.12 upper=0.77 effort=40 velocity=16.8; origin xyz=-0.1651 0.0115 -0.12977 rpy=0 0 0 -> xyz=0.1651 -0.12977 0.0115 rpy=3.141592653589793 0 0
- joint rfwheel: axis 0 -1 0 -> 0 0 1; limit lower=0 upper=0 effort=0 velocity=0 -> effort=3.9 velocity=58.4; origin xyz=0.1651 0.028 -0.18773 rpy=0 0 0 -> xyz=-0.1651 0.18773 -0.028 rpy=0 0 0

Commit message: 新增 chuanliantui 训练环境:照复旦 plane 方案跑通 train/play/sim2sim 全链
- envs/chuanliantui:env 子类仅覆写 FK 零位偏置(0.666151/1.625993),
  config 照复旦 plane 奖励/域随机化/指令课程,机器人参数换实值
  (l1=0.21/l2=0.25,站姿 ∓0.06/±0.10,站高 0.324m,DM8009P+改装M3508)
- 平地版 privileged 显式 67 维(measure_heights=False 时地形项塌缩)
- URDF mesh 路径 package:// 改 ../meshes/(Isaac 解析必需,动力学无变化)
- 新增 sim2sim/chuanliantui.xml(base 降面网格/mesh K 补偿旋转/轮解析圆柱)
  与 mj_sim2sim_ct.py(契约常量按 chuanliantui 改写,yaw=角速度直喂)

验收:model_5000 下 Isaac 内 cmd_vx=1 走 2.55m/3s 零终止;
MuJoCo 20s 不摔,速度跟踪至目标 6 成(5000 iter 短训水平)。
任务: T-20260823-01

Co-Authored-By: Claude Fable 5 <noreply@anthropic.com>

File: resources/robots/chuanliantui/urdf/chuanliantui.urdf (robot description, URDF)
Before this commit: robot chuanliantui, 7 links, 6 joints
Links:
- link base_link: geometry collision mesh filename=../meshes/base_link.STL; visual mesh filename=../meshes/base_link.STL
- link lf0: geometry collision mesh filename=../meshes/lf0.STL; visual mesh filename=../meshes/lf0.STL
- link lf1: geometry collision mesh filename=../meshes/lf1.STL; visual mesh filename=../meshes/lf1.STL
- link lfwheel: geometry collision mesh filename=../meshes/lfwheel.STL; visual mesh filename=../meshes/lfwheel.STL
- link rf0: geometry collision mesh filename=../meshes/rf0.STL; visual mesh filename=../meshes/rf0.STL
- link rf1: geometry collision mesh filename=../meshes/rf1.STL; visual mesh filename=../meshes/rf1.STL
- link rfwheel: geometry collision mesh filename=../meshes/rfwheel.STL; visual mesh filename=../meshes/rfwheel.STL
