Commit message: 修正串联腿闭链起立回放与膝关节限位
将原始 URDF 和闭链 XML 的左右膝限位对齐实机行程，并加入限位回归检查。
完善虚拟膝观测、力矩映射、Ctrl+R 复位和 Isaac 对照诊断，修复mujoco闭链问题。
收录起立训练的代码与配置快照、TensorBoard 日志及 model_6000 至 model_9000 权重。
记录 MuJoCo 起立回放结果及仍需实机验证的限制。

File: resources/robots/chuanliantui_new_1/urdf/chuanliantui.urdf (robot description, URDF)
Before this commit: robot chuanliantui, 24 links, 23 joints
Joints:
- joint lf1: limit lower=-0.77 upper=0.12 effort=0 velocity=0 -> lower=-0.12 upper=0.77 effort=0 velocity=0
- joint rf1: limit lower=-0.12 upper=0.77 effort=0 velocity=0 -> lower=-0.77 upper=0.12 effort=0 velocity=0

Commit message: 将串联腿训练迁移至 mjlab 并采用华南虎 V14 普通 PPO
新增独立 mjlab 训练、实体关节观测与控制、回放、验收和 ONNX 导出入口，移植华南虎 V14 flat v0 普通 PPO、奖励、延迟及域随机化逻辑。
修正 URDF 与 MuJoCo 资产左右命名并同步旧环境和适配脚本，依据 CAD 端点及轴向计算气弹簧随姿态变化的作用力。
补充依赖锁定、接口契约、命令与验证记录，完成奖励数值对照、CPU/GPU 有限物理及 ONNX 数值检查。
本次未启动训练或 TensorBoard，起立行为与 H7 实体接口适配仍待后续验证。

File: resources/robots/chuanliantui_new_1/urdf/chuanliantui.urdf (robot description, URDF)
Before this commit: robot chuanliantui, 24 links, 23 joints
Links:
- link lf0: geometry collision mesh filename=package://chuanliantui/meshes/rf0.STL; visual mesh filename=package://chuanliantui/meshes/rf0.STL
- link lf00: mass 0.108755464967074 -> 0.108755464967073; geometry collision mesh filename=package://chuanliantui/meshes/rf00.STL; visual mesh filename=package://chuanliantui/meshes/rf00.STL
- link lf001: mass 0.000125663706143592 -> 0.000125663706143591; geometry collision mesh filename=package://chuanliantui/meshes/rf001.STL; visual mesh filename=package://chuanliantui/meshes/rf001.STL
- link lf002: mass 0.000188495559215424 -> 0.000314159265358979; geometry collision mesh filename=package://chuanliantui/meshes/rf002.STL; visual mesh filename=package://chuanliantui/meshes/rf002.STL
- link lf01: mass 0.0527615983680122 -> 0.0527615983680123; geometry collision mesh filename=package://chuanliantui/meshes/rf01.STL; visual mesh filename=package://chuanliantui/meshes/rf01.STL
- link lf02: geometry collision mesh filename=package://chuanliantui/meshes/rf02.STL; visual mesh filename=package://chuanliantui/meshes/rf02.STL
- link lf03: mass 0.0511656410370526 -> 0.0511656410370527; geometry collision mesh filename=package://chuanliantui/meshes/rf03.STL; visual mesh filename=package://chuanliantui/meshes/rf03.STL
- link lf04: geometry collision mesh filename=package://chuanliantui/meshes/rf04.STL; visual mesh filename=package://chuanliantui/meshes/rf04.STL
- link lf05: geometry collision mesh filename=package://chuanliantui/meshes/rf05.STL; visual mesh filename=package://chuanliantui/meshes/rf05.STL
- link lf1: mass 0.414858418961741 -> 0.414858419057853; geometry collision mesh filename=package://chuanliantui/meshes/rf1.STL; visual mesh filename=package://chuanliantui/meshes/rf1.STL
- link lfwheel: mass 0.344781890910713 -> 0.344781890891785; geometry collision mesh filename=package://chuanliantui/meshes/rfwheel.STL; visual mesh filename=package://chuanliantui/meshes/rfwheel.STL
- link rf0: geometry collision mesh filename=package://chuanliantui/meshes/lf0.STL; visual mesh filename=package://chuanliantui/meshes/lf0.STL
- link rf00: mass 0.108755464967073 -> 0.108755464967074; geometry collision mesh filename=package://chuanliantui/meshes/lf00.STL; visual mesh filename=package://chuanliantui/meshes/lf00.STL
- link rf001: mass 0.000125663706143591 -> 0.000125663706143592; geometry collision mesh filename=package://chuanliantui/meshes/lf001.STL; visual mesh filename=package://chuanliantui/meshes/lf001.STL
- link rf002: mass 0.000314159265358979 -> 0.000188495559215424; geometry collision mesh filename=package://chuanliantui/meshes/lf002.STL; visual mesh filename=package://chuanliantui/meshes/lf002.STL
- link rf01: mass 0.0527615983680123 -> 0.0527615983680122; geometry collision mesh filename=package://chuanliantui/meshes/lf01.STL; visual mesh filename=package://chuanliantui/meshes/lf01.STL
- link rf02: geometry collision mesh filename=package://chuanliantui/meshes/lf02.STL; visual mesh filename=package://chuanliantui/meshes/lf02.STL
- link rf03: mass 0.0511656410370527 -> 0.0511656410370526; geometry collision mesh filename=package://chuanliantui/meshes/lf03.STL; visual mesh filename=package://chuanliantui/meshes/lf03.STL
- link rf04: geometry collision mesh filename=package://chuanliantui/meshes/lf04.STL; visual mesh filename=package://chuanliantui/meshes/lf04.STL
- link rf05: geometry collision mesh filename=package://chuanliantui/meshes/lf05.STL; visual mesh filename=package://chuanliantui/meshes/lf05.STL
- link rf1: mass 0.414858419057853 -> 0.414858418961741; geometry collision mesh filename=package://chuanliantui/meshes/lf1.STL; visual mesh filename=package://chuanliantui/meshes/lf1.STL
- link rfwheel: mass 0.344781890891785 -> 0.344781890910713; geometry collision mesh filename=package://chuanliantui/meshes/lfwheel.STL; visual mesh filename=package://chuanliantui/meshes/lfwheel.STL
Joints:
- joint lf0: axis 0 -1 0 -> 0 1 0; origin xyz=-0.0114000000001232 -0.178572975540517 0.0235199999997 rpy=0 0 0 -> xyz=-0.0114000000001256 0.176932975540448 0.0235200000001889 rpy=0 0 0
- joint lf00: axis 0 -1 0 -> 0 1 0; origin xyz=-0.0114000000001247 -0.189595000000041 0.023519999999691 rpy=0 0 0 -> xyz=-0.0114000000001251 0.18795499999997 0.0235200000002041 rpy=0 0 0
- joint lf001: axis 0 -1 0 -> 0 1 0; origin xyz=0.014206057708 -0.175072975540468 -0.0135852989315572 rpy=0 0 0 -> xyz=0.0142060577080023 0.173432975540499 -0.0135852989310789 rpy=0 0 0
- joint lf002: axis 0 -1 0 -> 0 1 0; origin xyz=-0.156996167107749 -0.200072975540276 -0.150480600144982 rpy=0 0 0 -> xyz=-0.156996167107753 0.198432975540677 -0.150480600144429 rpy=0 0 0
- joint lf01: axis 0 -1 0 -> 0 1 0; origin xyz=0.0890545087133239 0.0110249999992321 -0.0702058008845904 rpy=0 0 0 -> xyz=0.0890545087133235 -0.0110249999999036 -0.0702058008844835 rpy=0 0 0
- joint lf02: axis 0 -1 0 -> 0 1 0; origin xyz=-0.0893008846007706 -0.0165000000010802 -0.101244022092578 rpy=0 0 0 -> xyz=-0.0893008846007715 0.0165000000001005 -0.101244022092738 rpy=0 0 0
- joint lf03: axis 0 -1 0 -> 0 1 0; origin xyz=-0.115541773105979 0.0130000000017961 0.163022939626841 rpy=0 0 0 -> xyz=-0.115541773105976 -0.0130000000002235 0.163022939626966 rpy=0 0 0
- joint lf04: axis 0 -1 0 -> 0 1 0; origin xyz=-0.100655914012723 -0.195069999999905 -0.0464295662160984 rpy=0 0 0 -> xyz=-0.100655914012724 0.193430000000029 -0.0464295662155702 rpy=0 0 0
- joint lf05: axis 0 -1 0 -> 0 1 0; origin xyz=-0.203220964633882 -0.182069999999905 -0.0444935508680955 rpy=0 0 0 -> xyz=-0.203220964633881 0.180430000000026 -0.0444935508676031 rpy=0 0 0
- joint lf1: axis 0 -1 0 -> 0 1 0; limit lower=-0.12 upper=0.77 effort=0 velocity=0 -> lower=-0.77 upper=0.12 effort=0 velocity=0; origin xyz=-0.165288729653418 -0.0115000000014235 -0.129536233732203 rpy=0 0 0 -> xyz=-0.165288729653417 0.0114999999999917 -0.129536233732335 rpy=0 0 0
- joint lfwheel: axis 0 -1 0 -> 0 1 0; origin xyz=0.16483247801054 -0.0280000000020713 -0.187963438447404 rpy=0 0 0 -> xyz=0.164832478009991 0.0199999999999965 -0.187963438447721 rpy=0 0 0
- joint rf0: axis 0 1 0 -> 0 -1 0; origin xyz=-0.0114000000001256 0.176932975540448 0.0235200000001889 rpy=0 0 0 -> xyz=-0.0114000000001232 -0.178572975540517 0.0235199999997 rpy=0 0 0
- joint rf00: axis 0 1 0 -> 0 -1 0; origin xyz=-0.0114000000001251 0.18795499999997 0.0235200000002041 rpy=0 0 0 -> xyz=-0.0114000000001247 -0.189595000000041 0.023519999999691 rpy=0 0 0
- joint rf001: axis 0 1 0 -> 0 -1 0; origin xyz=0.0142060577080023 0.173432975540499 -0.0135852989310789 rpy=0 0 0 -> xyz=0.014206057708 -0.175072975540468 -0.0135852989315572 rpy=0 0 0
- joint rf002: axis 0 1 0 -> 0 -1 0; origin xyz=-0.156996167107753 0.198432975540677 -0.150480600144429 rpy=0 0 0 -> xyz=-0.156996167107749 -0.200072975540276 -0.150480600144982 rpy=0 0 0
- joint rf01: axis 0 1 0 -> 0 -1 0; origin xyz=0.0890545087133235 -0.0110249999999036 -0.0702058008844835 rpy=0 0 0 -> xyz=0.0890545087133239 0.0110249999992321 -0.0702058008845904 rpy=0 0 0
- joint rf02: axis 0 1 0 -> 0 -1 0; origin xyz=-0.0893008846007715 0.0165000000001005 -0.101244022092738 rpy=0 0 0 -> xyz=-0.0893008846007706 -0.0165000000010802 -0.101244022092578 rpy=0 0 0
- joint rf03: axis 0 1 0 -> 0 -1 0; origin xyz=-0.115541773105976 -0.0130000000002235 0.163022939626966 rpy=0 0 0 -> xyz=-0.115541773105979 0.0130000000017961 0.163022939626841 rpy=0 0 0
- joint rf04: axis 0 1 0 -> 0 -1 0; origin xyz=-0.100655914012724 0.193430000000029 -0.0464295662155702 rpy=0 0 0 -> xyz=-0.100655914012723 -0.195069999999905 -0.0464295662160984 rpy=0 0 0
- joint rf05: axis 0 1 0 -> 0 -1 0; origin xyz=-0.203220964633881 0.180430000000026 -0.0444935508676031 rpy=0 0 0 -> xyz=-0.203220964633882 -0.182069999999905 -0.0444935508680955 rpy=0 0 0
- joint rf1: axis 0 1 0 -> 0 -1 0; limit lower=-0.77 upper=0.12 effort=0 velocity=0 -> lower=-0.12 upper=0.77 effort=0 velocity=0; origin xyz=-0.165288729653417 0.0114999999999917 -0.129536233732335 rpy=0 0 0 -> xyz=-0.165288729653418 -0.0115000000014235 -0.129536233732203 rpy=0 0 0
- joint rfwheel: axis 0 1 0 -> 0 -1 0; origin xyz=0.164832478009991 0.0199999999999965 -0.187963438447721 rpy=0 0 0 -> xyz=0.16483247801054 -0.0280000000020713 -0.187963438447404 rpy=0 0 0

File: resources/robots/chuanliantui_new_1/urdf/chuanliantui_train.urdf (robot description, URDF)
Before this commit: robot chuanliantui, 24 links, 23 joints
Links:
- link lf0: geometry collision mesh filename=../meshes/rf0.STL; visual mesh filename=../meshes/rf0.STL
- link lf00: mass 0.108755464967074 -> 0.108755464967073; geometry collision mesh filename=../meshes/rf00.STL; visual mesh filename=../meshes/rf00.STL
- link lf001: mass 0.000125663706143592 -> 0.000125663706143591; geometry collision mesh filename=../meshes/rf001.STL; visual mesh filename=../meshes/rf001.STL
- link lf002: mass 0.000188495559215424 -> 0.000314159265358979; geometry collision mesh filename=../meshes/rf002.STL; visual mesh filename=../meshes/rf002.STL
- link lf01: mass 0.0527615983680122 -> 0.0527615983680123; geometry collision mesh filename=../meshes/rf01.STL; visual mesh filename=../meshes/rf01.STL
- link lf02: geometry collision mesh filename=../meshes/rf02.STL; visual mesh filename=../meshes/rf02.STL
- link lf03: mass 0.0511656410370526 -> 0.0511656410370527; geometry collision mesh filename=../meshes/rf03.STL; visual mesh filename=../meshes/rf03.STL
- link lf04: geometry collision mesh filename=../meshes/rf04.STL; visual mesh filename=../meshes/rf04.STL
- link lf05: geometry collision mesh filename=../meshes/rf05.STL; visual mesh filename=../meshes/rf05.STL
- link lf1: mass 0.414858418961741 -> 0.414858419057853; geometry collision mesh filename=../meshes/rf1.STL; visual mesh filename=../meshes/rf1.STL
- link lfwheel: mass 0.344781890910713 -> 0.344781890891785; geometry collision mesh filename=../meshes/rfwheel.STL; visual mesh filename=../meshes/rfwheel.STL
- link rf0: geometry collision mesh filename=../meshes/lf0.STL; visual mesh filename=../meshes/lf0.STL
- link rf00: mass 0.108755464967073 -> 0.108755464967074; geometry collision mesh filename=../meshes/lf00.STL; visual mesh filename=../meshes/lf00.STL
- link rf001: mass 0.000125663706143591 -> 0.000125663706143592; geometry collision mesh filename=../meshes/lf001.STL; visual mesh filename=../meshes/lf001.STL
- link rf002: mass 0.000314159265358979 -> 0.000188495559215424; geometry collision mesh filename=../meshes/lf002.STL; visual mesh filename=../meshes/lf002.STL
- link rf01: mass 0.0527615983680123 -> 0.0527615983680122; geometry collision mesh filename=../meshes/lf01.STL; visual mesh filename=../meshes/lf01.STL
- link rf02: geometry collision mesh filename=../meshes/lf02.STL; visual mesh filename=../meshes/lf02.STL
- link rf03: mass 0.0511656410370527 -> 0.0511656410370526; geometry collision mesh filename=../meshes/lf03.STL; visual mesh filename=../meshes/lf03.STL
- link rf04: geometry collision mesh filename=../meshes/lf04.STL; visual mesh filename=../meshes/lf04.STL
- link rf05: geometry collision mesh filename=../meshes/lf05.STL; visual mesh filename=../meshes/lf05.STL
- link rf1: mass 0.414858419057853 -> 0.414858418961741; geometry collision mesh filename=../meshes/lf1.STL; visual mesh filename=../meshes/lf1.STL
- link rfwheel: mass 0.344781890891785 -> 0.344781890910713; geometry collision mesh filename=../meshes/lfwheel.STL; visual mesh filename=../meshes/lfwheel.STL
Joints:
- joint lf0: axis 0 -1 0 -> 0 1 0; origin xyz=-0.0114000000001232 -0.178572975540517 0.0235199999997 rpy=0 0 0 -> xyz=-0.0114000000001256 0.176932975540448 0.0235200000001889 rpy=0 0 0
- joint lf00: origin xyz=-1.49880108324396e-15 -0.011022024459524 -8.99974539336768e-15 rpy=0 -0 0 -> xyz=4.9960036108132e-16 0.011022024459522 1.51996470965088e-14 rpy=0 -0 0
- joint lf001: origin xyz=0.014206057708 -0.175072975540468 -0.0135852989315572 rpy=0 0 0 -> xyz=0.0142060577080023 0.173432975540499 -0.0135852989310789 rpy=0 0 0
- joint lf002: origin xyz=-0.156996167107749 -0.200072975540276 -0.150480600144982 rpy=0 0 0 -> xyz=-0.156996167107753 0.198432975540677 -0.150480600144429 rpy=0 0 0
- joint lf01: origin xyz=0.0890545087133239 0.0110249999992321 -0.0702058008845904 rpy=0 -0 0 -> xyz=0.0890545087133235 -0.0110249999999036 -0.0702058008844835 rpy=0 -0 0
- joint lf02: origin xyz=-0.0893008846007706 -0.0165000000010802 -0.101244022092578 rpy=0 -0 0 -> xyz=-0.0893008846007715 0.0165000000001005 -0.101244022092738 rpy=0 -0 0
- joint lf03: origin xyz=-0.115541773105979 0.0130000000017961 0.163022939626841 rpy=0 -0 0 -> xyz=-0.115541773105976 -0.0130000000002235 0.163022939626966 rpy=0 -0 0
- joint lf04: origin xyz=-0.100655914012723 -0.195069999999905 -0.0464295662160984 rpy=0 0 0 -> xyz=-0.100655914012724 0.193430000000029 -0.0464295662155702 rpy=0 0 0
- joint lf05: origin xyz=-0.203220964633882 -0.182069999999905 -0.0444935508680955 rpy=0 0 0 -> xyz=-0.203220964633881 0.180430000000026 -0.0444935508676031 rpy=0 0 0
- joint lf1: axis 0 -1 0 -> 0 1 0; limit lower=-0.12 upper=0.77 effort=40 velocity=16.8 -> lower=-0.77 upper=0.12 effort=40 velocity=16.8; origin xyz=-0.165288729653418 -0.0115000000014235 -0.129536233732203 rpy=0 0 0 -> xyz=-0.165288729653417 0.0114999999999917 -0.129536233732335 rpy=0 0 0
- joint lfwheel: axis 0 -1 0 -> 0 1 0; origin xyz=0.16483247801054 -0.0280000000020713 -0.187963438447404 rpy=0 0 0 -> xyz=0.164832478009991 0.0199999999999965 -0.187963438447721 rpy=0 0 0
- joint rf0: axis 0 1 0 -> 0 -1 0; origin xyz=-0.0114000000001256 0.176932975540448 0.0235200000001889 rpy=0 0 0 -> xyz=-0.0114000000001232 -0.178572975540517 0.0235199999997 rpy=0 0 0
- joint rf00: origin xyz=4.9960036108132e-16 0.011022024459522 1.51996470965088e-14 rpy=0 -0 0 -> xyz=-1.49880108324396e-15 -0.011022024459524 -8.99974539336768e-15 rpy=0 -0 0
- joint rf001: origin xyz=0.0142060577080023 0.173432975540499 -0.0135852989310789 rpy=0 0 0 -> xyz=0.014206057708 -0.175072975540468 -0.0135852989315572 rpy=0 0 0
- joint rf002: origin xyz=-0.156996167107753 0.198432975540677 -0.150480600144429 rpy=0 0 0 -> xyz=-0.156996167107749 -0.200072975540276 -0.150480600144982 rpy=0 0 0
- joint rf01: origin xyz=0.0890545087133235 -0.0110249999999036 -0.0702058008844835 rpy=0 -0 0 -> xyz=0.0890545087133239 0.0110249999992321 -0.0702058008845904 rpy=0 -0 0
- joint rf02: origin xyz=-0.0893008846007715 0.0165000000001005 -0.101244022092738 rpy=0 -0 0 -> xyz=-0.0893008846007706 -0.0165000000010802 -0.101244022092578 rpy=0 -0 0
- joint rf03: origin xyz=-0.115541773105976 -0.0130000000002235 0.163022939626966 rpy=0 -0 0 -> xyz=-0.115541773105979 0.0130000000017961 0.163022939626841 rpy=0 -0 0
- joint rf04: origin xyz=-0.100655914012724 0.193430000000029 -0.0464295662155702 rpy=0 0 0 -> xyz=-0.100655914012723 -0.195069999999905 -0.0464295662160984 rpy=0 0 0
- joint rf05: origin xyz=-0.203220964633881 0.180430000000026 -0.0444935508676031 rpy=0 0 0 -> xyz=-0.203220964633882 -0.182069999999905 -0.0444935508680955 rpy=0 0 0
- joint rf1: axis 0 1 0 -> 0 -1 0; limit lower=-0.77 upper=0.12 effort=40 velocity=16.8 -> lower=-0.12 upper=0.77 effort=40 velocity=16.8; origin xyz=-0.165288729653417 0.0114999999999917 -0.129536233732335 rpy=0 0 0 -> xyz=-0.165288729653418 -0.0115000000014235 -0.129536233732203 rpy=0 0 0
- joint rfwheel: axis 0 1 0 -> 0 -1 0; origin xyz=0.164832478009991 0.0199999999999965 -0.187963438447721 rpy=0 0 0 -> xyz=0.16483247801054 -0.0280000000020713 -0.187963438447404 rpy=0 0 0
